File: TTRus.kicad_pcb (KiCad board)
At the start: 2 copper layers, 79.5 x 80.5 mm, 1 part

Commit message: Add files via upload
Parts:
- removed REF**: UAEFI_BRD, Hellen:uaefi
- added M1: Module:uaefi/0.2, Hellen:uaefi, F.Cu at (89.1, 143.9)

Commit message: Add files via upload
Parts:
- added J1: Screw_Terminal_01x20, TerminalBlock:TerminalBlock_Xinya_XY308-2.54-20P_1x20_P2.54mm_Horizontal, F.Cu at (204.5, 49.5)
Connections:
- M1 pad A4: unconnected-(M1-GND-PadA4) -> Net-(J1-Pin_3)
- M1 pad A7: unconnected-(M1-IN_VIGN-PadA7) -> Net-(J1-Pin_2)
- M1 pad A8: unconnected-(M1-IN_V_MAIN-PadA8) -> Net-(J1-Pin_1)
- M1 pad B15: unconnected-(M1-OUT_IGN1-PadB15) -> Net-(J1-Pin_3)
Routing:
- net Net-(J1-Pin_2): track 0.00 -> 243.0 mm
- net Net-(J1-Pin_1): track 0.00 -> 222.5 mm
- net Net-(J1-Pin_3): track 0.00 -> 154.9 mm
Other:
- board size 79.5 x 80.5 mm -> 135 x 105 mm
